File: hardware/dt_devboard/dt_devboard.kicad_sch (KiCad schematic)
At the start: 33 parts, among them IC1 MIMXRT1015CAF4A, IC2 ESP32-C3, Y1 Crystal_GND24

Commit message: added processor-specific design file
Connections:
- net U0RXD is gone; now on net UART2_TXD: IC2.27 (U0RXD)
- net U0TXD is gone; now on net UART2_TXD: R2.1
- net UART2_RXD: now reaches IC1.90 (GPIO_EMC_23)
- net UART2_TXD: now reaches IC1.93 (GPIO_EMC_22)
- net UART2_RTS_B: now reaches IC1.94 (GPIO_EMC_21)
- net UART2_CTS_B: now reaches IC1.96 (GPIO_EMC_20)
- net SIP1_SDO renamed SPI1_SDO
Other:
- note added: "UART connection between ESP32 and processor"
- moved on the sheet: C1, C10, C11, C12, C13, C14, C2, C3, C4, C5, C6, C7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
